File: kicad/cbpi_hat/hat.kicad_sch (KiCad schematic)
At the start: 25 parts, among them J1 GPIO, U1 CAT24C256

Commit message: Assigned all footprints to the DC DC converter
Parts:
- C1: footprint (none) -> Capacitor_SMD:C_0603_1608Metric
- C10: renamed from C?; footprint (none) -> Capacitor_SMD:C_Elec_6.3x5.4
- C2, C3: renamed from C?; footprint (none) -> Capacitor_SMD:C_1206_3216Metric
- C4, C5, C8, C9: renamed from C?; footprint (none) -> Capacitor_SMD:C_0603_1608Metric
- C6, C7: renamed from C?; footprint (none) -> Capacitor_SMD:C_0805_2012Metric
- L1: renamed from L?; footprint (none) -> SMMS1050-330M:IND-SMD_L11.5-W10.0
- R3, R4: renamed from R?; footprint (none) -> Resistor_SMD:R_0402_1005Metric
- R5, R6, R7, R8: renamed from R?; footprint (none) -> Resistor_SMD:R_0603_1608Metric
- gave numbers to parts that had none: 3
Other:
- company: (none) -> Till Klocke
- moved on the sheet: C10, C2, C3, C4, C5, C6, C7, C8, C9, D1, D2, L1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

Commit message: Added gitignore so we don't checkin the kicad backups anymore
Parts:
- added J2: Screw_Terminal_01x02, symbol Connector:Screw_Terminal_01x02
- JP1: footprint (none) -> Jumper:SolderJumper-2_P1.3mm_Open_RoundedPad1.0x1.5mm
- R1, R2: footprint (none) -> Resistor_SMD:R_0402_1005Metric
- U1: footprint (none) -> Package_SO:SOIC-8-1EP_3.9x4.9mm_P1.27mm_EP2.29x3mm
Connections:
- net +24V: now also J2.2 (Pin_2)
- net GND: now also J2.1 (Pin_1)
- no-connect marks 4 -> 30
Other:
- note added: "Identity EEPROM"
- note added: "RPi Power Supply +5V"
